File: acoustic-piezodriver-board/_autosave-acoustic-piezodriver-board.kicad_sch (KiCad schematic)
At the start: 5 parts, among them P101 WJ128V-5.0-3P, U101 AMS1117-3.3, U102 TMCS1108A3UQDR

Commit message: completed positioning (next) routing
Connections:
- net at P101.3, U102.1 (IN+), U102.2 (IN+): now also P101.2
Changed lines of the file:
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@@
+	)
+	(junction
+		(at 100.33 85.09)
+		(diameter 0)
+		(color 0 0 0 0)
 	)
 	(junction
@@
 		)
 		(stroke
+			(width 0)
+			(type default)
+		)
+	)
+	(wire
+		(pts
+			(xy 100.33 82.55) (xy 100.33 85.09)
+		)
+		(stroke
