File: acoustic-piezodriver-board/inverter.kicad_sch (KiCad schematic)
At the start: 42 parts, among them P201 WJ128V-5.0-3P, U201 UCC27282DR, U202 UCC27282DR, U204 TMCS1108A3UQDR, U6 NCE6005AS, U7 NCE6005AS

Commit message: changed footprints,  changed stackup from L3:PWR-> L3:GND and routed +BATT on 4th layer
Connections:
- net 10V renamed +10V
Other:
- sheet INVERTER_POWER ports: added +10V; removed 10V
Changed lines of the file:
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@@
 		)
 	)
-	(label "10V"
+	(label "+10V"
 		(at 120.65 30.48 180)
 		(effects
@@
 		)
 	)
-	(label "10V"
+	(label "+10V"
 		(at 349.25 27.94 180)
 		(effects
@@
 	)
 	(symbol
+		(lib_name "NCE6005AS_1")
 		(lib_id "custom_mosfet:NCE6005AS")
 		(at 252.73 90.17 0)
@@
 		(on_board yes)
 		(dnp no)
-		(fields_autoplaced yes)
 		(property "Reference" "U6"
-			(at 256.54 88.8999 0)
+			(at 253.492 93.218 0)
 			(effects
 				(font
@@
 		)
 		(property "Value" "NCE6005AS"
-			(at 256.54 91.4399 0)
+			(at 251.968 86.868 0)
 			(effects
 				(font
@@
 				)
 				(justify left)
+				(hide yes)
 			)
 		)
@@
 	)
 	(symbol
+		(lib_name "NCE6005AS_2")
 		(lib_id "custom_mosfet:NCE6005AS")
 		(at 252.73 110.49 0)
@@
 				)
 				(justify left)
+				(hide yes)
 			)
 		)
@@
 			)
 		)
-		(pin "10V" bidirectional
+		(pin "+10V" bidirectional
 			(at 341.63 33.02 90)
 			(effects

Commit message: [production checks] checked caps, [todo] Think about replacing 220 nF filtering caps in DC-DC to 0402 package (next) check rest of footprints
Parts:
- C1, C2: LCSC Part Number C5378 -> (none); LPN (none) -> C5378; MPN (none) -> CL21B224KBFNNNE; Manufacturing Part Number CL21B224KBFNNNE -> (none)
- C10, C12: LCSC Part Number C15195 -> (none); LPN (none) -> C15195; MPN (none) -> CL05B103KB5NNNC; Manufacturing Part Number CL05B103KB5NNNC -> (none)
- C11, C6, C8, C9: LCSC Part Number C15195 -> (none); LPN (none) -> C15195; MPN (none) -> CL05B103KB5NNNC
- C201, C202, C203: LCSC Part Number C2983797 -> (none); LPN (none) -> C2983797; MPN (none) -> SPZ1JM221G15O00RAXXX; Manufacturing Part Number SPZ1JM221G15O00RAXXX -> (none)
- C204, C205, C206, C207, C208, C209, C211, C212, C3, C4: LCSC Part Number C28323 -> (none); LPN (none) -> C28323; MPN (none) -> CL21B105KBFNNNE; Manufacturing Part Number CL21B105KBFNNNE -> (none)
- R1, R2, R3, R4: LCSC Part Number C17903 -> (none); LPN (none) -> C17903; MPN (none) -> 1206W4F100JT5E; Manufacturing Part Number 1206W4F100JT5E -> (none)
- R10, R5, R6, R7, R8, R9: LCSC Part Number C22936 -> (none); LPN (none) -> C22936; MPN (none) -> 0603WAF100KT5E; Manufacturing Part Number 0603WAF100KT5E -> (none)
- U201, U202: LCSC Part Number C2867844 -> (none); LPN (none) -> C2867844
- U7: LPN (none) -> C126151

Commit message: completed footprint check (next) reroute pbootstrap circuit on top layer only, fix errors after footprint change
Parts:
- U201, U202: footprint Package_SO:SOIC-8-1EP_3.9x4.9mm_P1.27mm_EP2.29x3mm -> Package_SO:SOIC-8_3.9x4.9mm_P1.27mm
Other:
- note added: "- Io: 0.74 A (R_gate: 1 ohm, R_fet: 10 ohm, 8-10 V Vhigh) - Q_gate: 22e-9 - 22e-9 / 0.74 = 30e-9s = 30 ns [100 ns period, 10 MHz], [1 us period, 1 MHz]"
Changed lines of the file:
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@@
 		)
 	)
+	(text "- Io: 0.74 A (R_gate: 1 ohm, R_fet: 10 ohm, 8-10 V Vhigh)\n- Q_gate: 22e-9\n	- 22e-9 / 0.74 = 30e-9s = 30 ns [100 ns period, 10 MHz], [1 us period, 1 MHz]"
+		(exclude_from_sim no)
+		(at 40.132 -13.208 0)
+		(effects
+			(font
+				(size 2.54 2.54)
+				(thickness 0.3175)
+			)
+			(justify left)
+		)
+	)
 	(text "DECOUPLING AND BULK"
 		(exclude_from_sim no)
@@
 		(dnp no)
 		(property "Reference" "R4"
-			(at 101.6 104.902 0)
+			(at 99.06 101.346 90)
 			(effects
 				(font
@@
 			)
 		)
-		(property "Description" "Resistor, small symbol"
+		(property "Description" "250mW"
 			(at 100.33 102.87 0)
 			(effects
@@
 			)
 		)
-		(property "Footprint" "Package_SO:SOIC-8-1EP_3.9x4.9mm_P1.27mm_EP2.29x3mm"
+		(property "Footprint" "Package_SO:SOIC-8_3.9x4.9mm_P1.27mm"
 			(at 86.36 73.406 0)
 			(effects
@@
 			)
 		)
-		(property "Description" "Resistor, small symbol"
+		(property "Description" "250mW"
 			(at 236.22 106.68 0)
 			(effects
@@
 			)
 		)
-		(property "Footprint" "Package_SO:SOIC-8-1EP_3.9x4.9mm_P1.27mm_EP2.29x3mm"
+		(property "Footprint" "Package_SO:SOIC-8_3.9x4.9mm_P1.27mm"
 			(at 210.82 74.93 0)
 			(effects
@@
 			)
 		)
-		(property "Description" "Resistor, small symbol"
+		(property "Description" "250mW"
 			(at 99.06 80.01 0)
 			(effects

Commit message: fixed erc and drc errors completely, added 3d models for connectors, finished DFM (next) create gerbers, check
Parts:
- U201, U202: footprint Package_SO:SOIC-8_3.9x4.9mm_P1.27mm -> Package_SO:SOIC-8-1EP_3.9x4.9mm_P1.27mm_EP2.29x3mm; LCSC Part Number (none) -> C2867844
Connections:
- net GND: no longer U201.9 (VSS), U202.9 (VSS)
Other:
- moved on the sheet: D8
Changed lines of the file:
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@@
 	)
 	(junction
-		(at 87.63 86.36)
-		(diameter 0)
-		(color 0 0 0 0)
-	)
-	(junction
 		(at 184.15 58.42)
 		(diameter 0)
@@
 	)
 	(junction
+		(at 87.63 87.63)
+		(diameter 0)
+		(color 0 0 0 0)
+	)
+	(junction
 		(at 257.81 57.15)
 		(diameter 0)
@@
 	(wire
 		(pts
-			(xy 102.87 86.36) (xy 107.95 86.36)
+			(xy 102.87 88.9) (xy 107.95 88.9)
 		)
 		(stroke
@@
 	(wire
 		(pts
-			(xy 107.95 81.28) (xy 107.95 86.36)
+			(xy 107.95 81.28) (xy 107.95 88.9)
 		)
 		(stroke
@@
 	(wire
 		(pts
-			(xy 87.63 86.36) (xy 95.25 86.36)
+			(xy 87.63 88.9) (xy 87.63 87.63)
+		)
+		(stroke
+			(width 0)
+			(type default)
+		)
+	)
+	(wire
+		(pts
+			(xy 87.63 88.9) (xy 95.25 88.9)
 		)
 		(stroke
@@
 	(wire
 		(pts
-			(xy 87.63 86.36) (xy 87.63 87.63)
+			(xy 87.63 80.01) (xy 87.63 87.63)
 		)
 		(stroke
@@
 	(wire
 		(pts
-			(xy 87.63 80.01) (xy 87.63 86.36)
-		)
-		(stroke
-			(width 0)
-			(type default)
-		)
-	)
-	(wire
-		(pts
 			(xy 242.57 90.17) (xy 242.57 85.09)
 		)
@@
 	)
 	(symbol
+		(lib_name "UCC27282DR_1")
 		(lib_id "iw-power:UCC27282DR")
 		(at 74.93 92.71 0)
@@
 			)
 		)
-		(property "Footprint" "Package_SO:SOIC-8_3.9x4.9mm_P1.27mm"
+		(property "Footprint" "Package_SO:SOIC-8-1EP_3.9x4.9mm_P1.27mm_EP2.29x3mm"
 			(at 86.36 73.406 0)
 			(effects
@@
 			)
 		)
+		(property "LCSC Part Number" "C2867844"
+			(at 74.93 92.71 0)
+			(effects
+				(font
+					(size 1.27 1.27)
+				)
+				(hide yes)
+			)
+		)
 		(pin "6"
 		)
@@
 		(pin "1"
 		)
-		(pin "9"
-		)
 		(instances
 			(project "acoustic-piezodriver-board"
@@
 	(symbol
 		(lib_id "Diode:SS14")
-		(at 99.06 86.36 0)
+		(at 99.06 88.9 0)
 		(unit 1)
 		(exclude_from_sim no)
@@
 		(dnp no)
 		(property "Reference" "D8"
-			(at 94.742 87.63 0)
+			(at 94.742 90.17 0)
 			(effects
 				(font
@@
 		)
 		(property "Value" "SS14"
-			(at 103.124 87.63 0)
+			(at 103.124 90.17 0)
 			(effects
 				(font
@@
 		)
 		(property "Footprint" "Diode_SMD:D_SMA"
-			(at 99.06 90.805 0)
+			(at 99.06 93.345 0)
 			(effects
 				(font
@@
 		)
 		(property "Datasheet" "https://www.vishay.com/docs/88746/ss12.pdf"
-			(at 99.06 86.36 0)
+			(at 99.06 88.9 0)
 			(effects
 				(font
@@
 		)
 		(property "Description" "40V 1A Schottky Diode, SMA"
-			(at 99.06 86.36 0)
+			(at 99.06 88.9 0)
 			(effects
 				(font
@@
 		)
 		(property "LPN" "C2480"
-			(at 99.06 86.36 0)
+			(at 99.06 88.9 0)
 			(effects
 				(font
@@
 		)
 		(property "MPN" "SS14"
-			(at 99.06 86.36 0)
+			(at 99.06 88.9 0)
 			(effects
 				(font
@@
 			)
 		)
-		(property "Footprint" "Package_SO:SOIC-8_3.9x4.9mm_P1.27mm"
+		(property "Footprint" "Package_SO:SOIC-8-1EP_3.9x4.9mm_P1.27mm_EP2.29x3mm"
 			(at 210.82 74.93 0)
 			(effects
@@
 			)
 		)
+		(property "LCSC Part Number" "C2867844"
+			(at 210.82 95.25 0)
+			(effects
+				(font
+					(size 1.27 1.27)
+				)
+				(hide yes)
+			)
+		)
 		(pin "6"
 		)
@@
 		(pin "1"
 		)
-		(pin "9"
-		)
 		(instances

Commit message: added testpoints on fb and isense pins (next) double-check schematic and order
Parts:
- C1, C2: LCSC Part Number (none) -> C5378; LPN C5378 -> (none); MPN CL21B224KBFNNNE -> (none); Manufacturing Part Number (none) -> CL21B224KBFNNNE
- C10, C11, C12, C6, C8, C9: LCSC Part Number (none) -> C15195; LPN C15195 -> (none); MPN CL05B103KB5NNNC -> (none); Manufacturing Part Number (none) -> CL05B103KB5NNNC
- C201, C202, C203: LCSC Part Number (none) -> C2983797; LPN C2983797 -> (none); MPN SPZ1JM221G15O00RAXXX -> (none); Manufacturing Part Number (none) -> SPZ1JM221G15O00RAXXX
- C204, C205, C206, C207, C208, C209, C211, C212, C3, C4: LCSC Part Number (none) -> C28323; LPN C28323 -> (none); MPN CL21B105KBFNNNE -> (none); Manufacturing Part Number (none) -> CL21B105KBFNNNE
- C210: LCSC Part Number (none) -> C307331; LPN C307331 -> (none); MPN CL05B104KB54PNC -> (none); Manufacturing Part Number (none) -> CL05B104KB54PNC
- D10, D11, D8, D9: LCSC Part Number (none) -> C2480; LPN C2480 -> (none); MPN SS14 -> (none); Manufacturing Part Number (none) -> SS14
- P201: LCSC Part Number (none) -> C8270; LPN C8270 -> (none); MPN WJ128V-5.0-3P -> (none); Manufacturing Part Number (none) -> WJ128V-5.0-3P
- R1, R2, R3, R4: LCSC Part Number (none) -> C17903; LPN C17903 -> (none); MPN 1206W4F100JT5E -> (none); Manufacturing Part Number (none) -> 1206W4F100JT5E
- R10, R5, R6, R7, R8, R9: LCSC Part Number (none) -> C22936; LPN C22936 -> (none); MPN 0603WAF100KT5E -> (none); Manufacturing Part Number (none) -> 0603WAF100KT5E
- U201, U202: footprint Package_SO:SOIC-8-1EP_3.9x4.9mm_P1.27mm_EP2.29x3mm -> Package_SO:SOIC-8_3.9x4.9mm_P1.27mm; LPN C2867844 -> (none); MPN UCC27282DR -> (none); Manufacturing Part Number (none) -> UCC27282DR
- U204: LCSC Part Number (none) -> C3684263; LPN C3684263 -> (none); MPN TMCS1108A3UQDR -> (none); Manufacturing Part Number (none) -> TMCS1108A3UQDR
- U6, U7: LCSC Part Number (none) -> C126151; LPN C126151 -> (none); MPN NCE6005AS -> (none); Manufacturing Part Number (none) -> NCE6005AS
