File: acoustic-piezodriver-board/sensor_conn.kicad_sch (KiCad schematic)
At the start: 26 parts, among them J501 Conn_02x06_Odd_Even, U402 TMP102xxDRL, U403 TMP102xxDRL, U404 ADS1115IDGS

Commit message: added testpoints on fb and isense pins (next) double-check schematic and order
Parts:
- C401, C403: LCSC Part Number (none) -> C15195; LPN C15195 -> (none); MPN CL05B103KB5NNNC -> (none); Manufacturing Part Number (none) -> CL05B103KB5NNNC
- C402, C405, C406: LCSC Part Number (none) -> C16772; LPN C16772 -> (none); MPN CL05B224KO5NNNC -> (none); Manufacturing Part Number (none) -> CL05B224KO5NNNC
- C404: LCSC Part Number (none) -> C307331; LPN C307331 -> (none); MPN CL05B104KB54PNC -> (none); Manufacturing Part Number (none) -> CL05B104KB54PNC
- D401, D402: LCSC Part Number (none) -> C2286; LPN C2286 -> (none); MPN KT-0603R -> (none); Manufacturing Part Number (none) -> KT-0603R
- J501: LCSC Part Number (none) -> C124388; LPN C124388 -> (none); MPN B-2100S12P-B110 -> (none); Manufacturing Part Number (none) -> B-2100S12P-B110
- R401, R405, R409, R410, R414: LCSC Part Number (none) -> C11702; LPN C11702 -> (none); MPN 0402WGF1001TCE -> (none); Manufacturing Part Number (none) -> 0402WGF1001TCE
- R402, R406: LCSC Part Number (none) -> C15402; LPN C15402 -> (none); MPN 0603WAJ0000T5E -> (none); Manufacturing Part Number (none) -> 0603WAJ0000T5E
- R403, R404: LCSC Part Number (none) -> C25900; LPN C25900 -> (none); MPN 0402WGF4701TCE -> (none); Manufacturing Part Number (none) -> 0402WGF4701TCE
- R407, R408, R411: LCSC Part Number (none) -> C15401; LPN C15401 -> (none); MPN 0603WAJ0103T5E -> (none); Manufacturing Part Number (none) -> 0603WAJ0103T5E
- R412: LCSC Part Number (none) -> C4177; LPN C4177 -> (none); MPN 0603WAF1801T5E -> (none); Manufacturing Part Number (none) -> 0603WAF1801T5E
- R413: LCSC Part Number (none) -> C25765; LPN C25765 -> (none); MPN 0402WGF2002TCE -> (none); Manufacturing Part Number (none) -> 0402WGF2002TCE
- U402, U403: LCSC Part Number (none) -> C99269; LPN C99269 -> (none); MPN TMP102AIDRLR -> (none); Manufacturing Part Number (none) -> TMP102AIDRLR
- U404: LCSC Part Number (none) -> C37593; LPN C37593 -> (none); MPN ADS1115IDGSR -> (none); Manufacturing Part Number (none) -> ADS1115IDGSR
Changed lines of the file:
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@@
 			)
 		)
-		(property "MPN" "0402WGF1001TCE"
+		(property "LCSC Part Number" "C11702"
 			(at 158.75 220.98 90)
 			(effects
@@
 			)
 		)
-		(property "LPN" "C11702"
+		(property "Manufacturing Part Number" "0402WGF1001TCE"
 			(at 158.75 220.98 90)
 			(effects
@@
 			)
 		)
-		(property "MPN" "0402WGF1001TCE"
-			(at 81.28 90.17 90)
+		(property "LCSC Part Number" "C11702"
+			(at 81.28 90.17 0)
 			(effects
 				(font
@@
 			)
 		)
-		(property "LPN" "C11702"
-			(at 81.28 90.17 90)
+		(property "Manufacturing Part Number" "0402WGF1001TCE"
+			(at 81.28 90.17 0)
 			(effects
 				(font
@@
 			)
 		)
-		(property "MPN" "0402WGF1001TCE"
-			(at 82.55 49.53 90)
+		(property "LCSC Part Number" "C11702"
+			(at 82.55 49.53 0)
 			(effects
 				(font
@@
 			)
 		)
-		(property "LPN" "C11702"
-			(at 82.55 49.53 90)
+		(property "Manufacturing Part Number" "0402WGF1001TCE"
+			(at 82.55 49.53 0)
 			(effects
 				(font
@@
 			)
 		)
-		(property "LPN" "C15195"
+		(property "LCSC Part Number" "C15195"
 			(at 73.66 49.53 0)
 			(effects
@@
 			)
 		)
-		(property "MPN" "CL05B103KB5NNNC"
+		(property "Manufacturing Part Number" "CL05B103KB5NNNC"
 			(at 73.66 49.53 0)
 			(effects
@@
 			)
 		)
-		(property "LPN" "C124388"
+		(property "LCSC Part Number" "C124388"
 			(at 152.4 101.6 0)
 			(effects
@@
 			)
 		)
-		(property "MPN" "B-2100S12P-B110 "
+		(property "Manufacturing Part Number" "B-2100S12P-B110 "
 			(at 152.4 101.6 0)
 			(effects
@@
 			)
 		)
-		(property "LPN" "C2286"
+		(property "LCSC Part Number" "C2286"
 			(at 82.55 55.88 0)
 			(effects
@@
 			)
 		)
-		(property "MPN" "KT-0603R "
+		(property "Manufacturing Part Number" "KT-0603R "
 			(at 82.55 55.88 0)
 			(effects
@@
 			)
 		)
-		(property "LPN" "C15401"
+		(property "LCSC Part Number" "C15401"
 			(at 86.36 203.2 90)
 			(effects
@@
 			)
 		)
-		(property "MPN" "0603WAJ0103T5E"
+		(property "Manufacturing Part Number" "0603WAJ0103T5E"
 			(at 86.36 203.2 90)
 			(effects
@@
 			)
 		)
-		(property "LPN" "C16772"
+		(property "LCSC Part Number" "C16772"
 			(at 153.67 173.99 0)
 			(effects
@@
 			)
 		)
-		(property "MPN" "CL05B224KO5NNNC"
+		(property "Manufacturing Part Number" "CL05B224KO5NNNC"
 			(at 153.67 173.99 0)
 			(effects
@@
 			)
 		)
-		(property "MPN" "0402WGF1001TCE"
+		(property "LCSC Part Number" "C11702"
 			(at 158.75 196.85 90)
 			(effects
@@
 			)
 		)
-		(property "LPN" "C11702"
+		(property "Manufacturing Part Number" "0402WGF1001TCE"
 			(at 158.75 196.85 90)
 			(effects
@@
 			)
 		)
-		(property "LPN" "C15402"
-			(at 52.07 106.68 90)
+		(property "LCSC Part Number" "C15402"
+			(at 52.07 106.68 0)
 			(effects
 				(font
@@
 			)
 		)
-		(property "MPN" "0603WAJ0000T5E"
-			(at 52.07 106.68 90)
+		(property "Manufacturing Part Number" "0603WAJ0000T5E"
+			(at 52.07 106.68 0)
 			(effects
 				(font
@@
 			)
 		)
-		(property "LPN" "C25900"
+		(property "LCSC Part Number" "C25900"
 			(at 92.71 74.93 90)
 			(effects
@@
 			)
 		)
-		(property "MPN" "0402WGF4701TCE"
+		(property "Manufacturing Part Number" "0402WGF4701TCE"
 			(at 92.71 74.93 90)
 			(effects
@@
 			)
 		)
-		(property "LPN" "C15401"
+		(property "LCSC Part Number" "C15401"
 			(at 54.61 115.57 90)
 			(effects
@@
 			)
 		)
-		(property "MPN" "0603WAJ0103T5E"
+		(property "Manufacturing Part Number" "0603WAJ0103T5E"
 			(at 54.61 115.57 90)
 			(effects
@@
 			)
 		)
-		(property "LPN" "C15402"
-			(at 48.26 55.88 90)
+		(property "LCSC Part Number" "C15402"
+			(at 48.26 55.88 0)
 			(effects
 				(font
@@
 			)
 		)
-		(property "MPN" "0603WAJ0000T5E"
-			(at 48.26 55.88 90)
+		(property "Manufacturing Part Number" "0603WAJ0000T5E"
+			(at 48.26 55.88 0)
 			(effects
 				(font
@@
 			)
 		)
-		(property "LPN" "C37593"
+		(property "LCSC Part Number" "C37593"
 			(at 101.6 194.31 0)
 			(effects
@@
 			)
 		)
-		(property "MPN" "ADS1115IDGSR"
+		(property "Manufacturing Part Number" "ADS1115IDGSR"
 			(at 101.6 194.31 0)
 			(effects
@@
 			)
 		)
-		(property "LPN" "C15401"
+		(property "LCSC Part Number" "C15401"
 			(at 49.53 72.39 90)
 			(effects
@@
 			)
 		)
-		(property "MPN" "0603WAJ0103T5E"
+		(property "Manufacturing Part Number" "0603WAJ0103T5E"
 			(at 49.53 72.39 90)
 			(effects
@@
 			)
 		)
-		(property "LPN" "C16772"
+		(property "LCSC Part Number" "C16772"
 			(at 153.67 200.66 0)
 			(effects
@@
 			)
 		)
-		(property "MPN" "CL05B224KO5NNNC"
+		(property "Manufacturing Part Number" "CL05B224KO5NNNC"
 			(at 153.67 200.66 0)
 			(effects
@@
 			)
 		)
-		(property "LPN" "C99269"
+		(property "LCSC Part Number" "C99269"
 			(at 69.85 64.77 0)
 			(effects
@@
 			)
 		)
-		(property "MPN" "TMP102AIDRLR"
+		(property "Manufacturing Part Number" "TMP102AIDRLR"
 			(at 69.85 64.77 0)
 			(effects
@@
 			)
 		)
-		(property "LPN" "C25765"
+		(property "LCSC Part Number" "C25765"
 			(at 255.27 96.52 0)
 			(effects
@@
 			)
 		)
-		(property "MPN" "0402WGF2002TCE"
+		(property "Manufacturing Part Number" "0402WGF2002TCE"
 			(at 255.27 96.52 0)
 			(effects
@@
 			)
 		)
-		(property "LPN" "C16772"
+		(property "LCSC Part Number" "C16772"
 			(at 153.67 224.79 0)
 			(effects
@@
 			)
 		)
-		(property "MPN" "CL05B224KO5NNNC"
+		(property "Manufacturing Part Number" "CL05B224KO5NNNC"
 			(at 153.67 224.79 0)
 			(effects
@@
 			)
 		)
-		(property "LPN" "C2286"
+		(property "LCSC Part Number" "C2286"
 			(at 81.28 96.52 0)
 			(effects
@@
 			)
 		)
-		(property "MPN" "KT-0603R "
+		(property "Manufacturing Part Number" "KT-0603R "
 			(at 81.28 96.52 0)
 			(effects
@@
 			)
 		)
-		(property "LPN" "C4177"
+		(property "LCSC Part Number" "C4177"
 			(at 255.27 107.95 0)
 			(effects
@@
 			)
 		)
-		(property "MPN" "0603WAF1801T5E"
+		(property "Manufacturing Part Number" "0603WAF1801T5E"
 			(at 255.27 107.95 0)
 			(effects
@@
 			)
 		)
-		(property "LPN" "C99269"
+		(property "LCSC Part Number" "C99269"
 			(at 68.58 105.41 0)
 			(effects
@@
 			)
 		)
-		(property "MPN" "TMP102AIDRLR"
+		(property "Manufacturing Part Number" "TMP102AIDRLR"
 			(at 68.58 105.41 0)
 			(effects
@@
 			)
 		)
-		(property "LPN" "C25900"
+		(property "LCSC Part Number" "C25900"
 			(at 104.14 74.93 90)
 			(effects
@@
 			)
 		)
-		(property "MPN" "0402WGF4701TCE"
+		(property "Manufacturing Part Number" "0402WGF4701TCE"
 			(at 104.14 74.93 90)
 			(effects
@@
 			)
 		)
-		(property "MPN" "0402WGF1001TCE"
+		(property "LCSC Part Number" "C11702"
 			(at 158.75 170.18 90)
 			(effects
@@
 			)
 		)
-		(property "LPN" "C11702"
+		(property "Manufacturing Part Number" "0402WGF1001TCE"
 			(at 158.75 170.18 90)
 			(effects
@@
 			)
 		)
-		(property "LPN" "C15195"
+		(property "LCSC Part Number" "C15195"
 			(at 72.39 90.17 0)
 			(effects
@@
 			)
 		)
-		(property "MPN" "CL05B103KB5NNNC"
+		(property "Manufacturing Part Number" "CL05B103KB5NNNC"
 			(at 72.39 90.17 0)
 			(effects
@@
 			)
 		)
-		(property "LPN" "C307331"
+		(property "LCSC Part Number" "C307331"
 			(at 110.49 177.8 0)
 			(effects
@@
 			)
 		)
-		(property "MPN" "CL05B104KB54PNC"
+		(property "Manufacturing Part Number" "CL05B104KB54PNC"
 			(at 110.49 177.8 0)
 			(effects
