File: acoustic-piezodriver-board/INVERTER_POWER.kicad_sch (KiCad schematic)
At the start: 62 parts, among them Q501 AO3400A, Q502 AO3400A, U501 NCE6005AS, U502 LM3478MM, U503 NCE6005AS, U504 LM3478MM

Commit message: added gerbers
Parts:
- TP503, TP504, TP505, TP506: now left out of the parts list
Other:
- note added: "DC-DC (Boost) VBAT -> 40 V - RDIV: 40 * (1 / 31) = 1.29 V - Capacitors here must be able to withstand 50 V - Compensation: Check notebook"
- note added: "FB RDIV: - 10 V * (0.68 / (0.68 + 4.7))) = 1.26 V"
- note removed: "Capacitors here must be able to withstand 50 V"
- note removed: "DC-DC (Boost) VBAT -> 40 V"
Changed lines of the file:
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@@
 		)
 	)
-	(text "DC-DC (Boost) VBAT -> 40 V"
+	(text "DC-DC (Boost) VBAT -> 40 V\n- RDIV: 40 * (1 / 31) = 1.29 V\n- Capacitors here must be able to withstand 50 V\n- Compensation: Check notebook"
 		(exclude_from_sim no)
-		(at 316.484 157.734 0)
+		(at 302.006 148.844 0)
 		(effects
 			(font
 				(size 1.27 1.27)
 			)
+			(justify left)
 		)
 	)
@@
 		)
 	)
-	(text "Capacitors here must be able to withstand 50 V"
+	(text "FB RDIV:\n- 10 V * (0.68 / (0.68 + 4.7))) = 1.26 V"
 		(exclude_from_sim no)
-		(at 305.054 164.846 0)
+		(at 283.718 116.332 0)
 		(effects
 			(font
@@
 		(unit 1)
 		(exclude_from_sim no)
-		(in_bom yes)
+		(in_bom no)
 		(on_board yes)
 		(dnp no)
@@
 		(unit 1)
 		(exclude_from_sim no)
-		(in_bom yes)
+		(in_bom no)
 		(on_board yes)
 		(dnp no)
@@
 		(unit 1)
 		(exclude_from_sim no)
-		(in_bom yes)
+		(in_bom no)
 		(on_board yes)
 		(dnp no)
@@
 		(unit 1)
 		(exclude_from_sim no)
-		(in_bom yes)
+		(in_bom no)
 		(on_board yes)
 		(dnp no)
